File: PHIIDXDP.kicad_pcb (KiCad board)
At the start: 2 copper layers, 0 parts

Commit message: symbol VOMIT
updated footprints and started PCB work lol
Parts:
- added C1: 1uF, Capacitor_SMD:C_0805_2012Metric, F.Cu at (19.0, 103.5)
- added C2: 0.1uf, Capacitor_SMD:C_0805_2012Metric, F.Cu at (19.0, 106.5)
- added C3: 0.1uf, Capacitor_SMD:C_0805_2012Metric, F.Cu at (19.0, 109.5)
- added C4: 0.1uf, Capacitor_SMD:C_0805_2012Metric, F.Cu at (19.0, 112.5)
- added C5: 10uf, Capacitor_SMD:C_0805_2012Metric, F.Cu at (19.0, 115.5)
- added C6: 22pF, Capacitor_SMD:C_0805_2012Metric, F.Cu at (19.0, 118.5)
- added C7: 22pF, Capacitor_SMD:C_0805_2012Metric, F.Cu at (19.0, 121.6)
- added F1: 500mA, Fuse:Fuse_1206_3216Metric, F.Cu at (49.6, 120.0)
- added J1: USB_C_Receptacle_USB2.0_16P, Connector_USB:USB_C_Receptacle_HRO_TYPE-C-31-M-12, F.Cu at (160.0, 18.5)
- added J10: 2P BT 2, Connector_JST:JST_XH_B4B-XH-AM_1x04_P2.50mm_Vertical, F.Cu at (187.0, 47.0)
- added J11: 2P BT 3, Connector_JST:JST_XH_B4B-XH-AM_1x04_P2.50mm_Vertical, F.Cu at (202.8, 36.5)
- added J12: 2P BT 4, Connector_JST:JST_XH_B4B-XH-AM_1x04_P2.50mm_Vertical, F.Cu at (203.0, 47.5)
- added J13: 2P BT 5, Connector_JST:JST_XH_B4B-XH-AM_1x04_P2.50mm_Vertical, F.Cu at (217.5, 36.5)
- added J14: 2P BT 6, Connector_JST:JST_XH_B4B-XH-AM_1x04_P2.50mm_Vertical, F.Cu at (217.5, 47.5)
- added J15: 2P BT 7, Connector_JST:JST_XH_B4B-XH-AM_1x04_P2.50mm_Vertical, F.Cu at (232.5, 36.5)
- added J16: 1P START, Connector_JST:JST_XH_B4B-XH-AM_1x04_P2.50mm_Vertical, F.Cu at (106.0, 19.0)
- added J17: EFFECT, Connector_JST:JST_XH_B4B-XH-AM_1x04_P2.50mm_Vertical, F.Cu at (125.5, 17.0)
- added J18: VEFX, Connector_JST:JST_XH_B4B-XH-AM_1x04_P2.50mm_Vertical, F.Cu at (177.5, 17.5)
- added J19: 2P START, Connector_JST:JST_XH_B4B-XH-AM_1x04_P2.50mm_Vertical, F.Cu at (195.5, 18.0)
- added J2: 1P BT 1, Connector_JST:JST_XH_B4B-XH-AM_1x04_P2.50mm_Vertical, F.Cu at (127.5, 35.5)
- added J20: P1 TT analog, Connector_JST:JST_XH_B3B-XH-AM_1x03_P2.50mm_Vertical, F.Cu at (68.5, 35.5)
- added J21: P2 TT analog, Connector_JST:JST_XH_B3B-XH-AM_1x03_P2.50mm_Vertical, F.Cu at (248.0, 36.5)
- added J22: LED P1 TT, Connector_JST:JST_XH_B3B-XH-AM_1x03_P2.50mm_Vertical, F.Cu at (113.5, 55.0)
- added J23: LED P2 TT, Connector_JST:JST_XH_B3B-XH-AM_1x03_P2.50mm_Vertical, F.Cu at (204.5, 57.0)
- added J24: LED P1 Buttons, Connector_JST:JST_XH_B3B-XH-AM_1x03_P2.50mm_Vertical, F.Cu at (129.5, 55.0)
- added J25: LED P2 Buttons, Connector_JST:JST_XH_B3B-XH-AM_1x03_P2.50mm_Vertical, F.Cu at (188.5, 56.0)
- added J26: LED CENTER, Connector_JST:JST_XH_B3B-XH-AM_1x03_P2.50mm_Vertical, F.Cu at (158.0, 34.5)
- added J28: P1 TT Encoder, Connector_JST:JST_XH_B4B-XH-AM_1x04_P2.50mm_Vertical, F.Cu at (82.5, 45.0)
- added J29: P2 TT Encoder, Connector_JST:JST_XH_B4B-XH-AM_1x04_P2.50mm_Vertical, F.Cu at (232.5, 47.5)
- added J3: 1P BT 3, Connector_JST:JST_XH_B4B-XH-AM_1x04_P2.50mm_Vertical, F.Cu at (112.5, 35.5)
- added J4: 1P BT 5, Connector_JST:JST_XH_B4B-XH-AM_1x04_P2.50mm_Vertical, F.Cu at (97.5, 35.5)
- added J5: 1P BT 7, Connector_JST:JST_XH_B4B-XH-AM_1x04_P2.50mm_Vertical, F.Cu at (82.5, 35.5)
- added J6: 1P BT 2, Connector_JST:JST_XH_B4B-XH-AM_1x04_P2.50mm_Vertical, F.Cu at (128.0, 45.0)
- added J7: 1P BT 4, Connector_JST:JST_XH_B4B-XH-AM_1x04_P2.50mm_Vertical, F.Cu at (113.0, 45.5)
- added J8: 1P BT 6, Connector_JST:JST_XH_B4B-XH-AM_1x04_P2.50mm_Vertical, F.Cu at (97.5, 45.5)
- added J9: 2P BT 1, Connector_JST:JST_XH_B4B-XH-AM_1x04_P2.50mm_Vertical, F.Cu at (187.2, 36.5)
- added R1: 10k, Resistor_SMD:R_0805_2012Metric, F.Cu at (26.9, 107.5)
- added R2: 22, Resistor_SMD:R_0805_2012Metric, F.Cu at (26.9, 110.5)
- added R3: 22, Resistor_SMD:R_0805_2012Metric, F.Cu at (26.9, 113.5)
- added R4: 10K, Resistor_SMD:R_0805_2012Metric, F.Cu at (26.9, 116.4)
- added R5: 5k1, Resistor_SMD:R_0805_2012Metric, F.Cu at (26.9, 119.3)
- added R6: 5k1, Resistor_SMD:R_0805_2012Metric, F.Cu at (26.9, 122.3)
- added SW1: SW_Push, Button_Switch_SMD:SW_SPST_SKQG_WithStem, F.Cu at (93.0, 78.5)
- added U1: AT90USB647-A, Package_QFP:TQFP-64_14x14mm_P0.8mm, F.Cu at (159.0, 90.5)
- added Y1: 16MHz, Crystal:Crystal_SMD_3225-4Pin_3.2x2.5mm, F.Cu at (84.4, 86.2)
