File: PHIIDXDP.kicad_pcb (KiCad board)
At the start: 2 copper layers, 45 parts, among them J1 USB_C_Receptacle_USB2.0_16P, J10 2P BT 2, J11 2P BT 3, J12 2P BT 4, J13 2P BT 5, J14 2P BT 6, J15 2P BT 7, J16 1P START, J17 EFFECT, J18 VEFX, J19 2P START, J2 1P BT 1, J20 P1 TT analog, J21 P2 TT analog, J22 LED P1 TT, J23 LED P2 TT, J24 LED P1 Buttons, J25 LED P2 Buttons, J26 LED CENTER, J28 P1 TT Encoder, J29 P2 TT Encoder, J3 1P BT 3, J4 1P BT 5, J5 1P BT 7, J6 1P BT 2, J7 1P BT 4, J8 1P BT 6, J9 2P BT 1, SW1 SW_Push, U1 AT90USB647-A, Y1 16MHz

Commit message: attempt at compacting connectors
Parts:
- moved J24 107.8 mm to (23.0, 38.0), turned to 90 degrees
- moved J22 90.6 mm to (23.0, 51.0), turned to 90 degrees
- moved U1 87.3 mm to (78.7, 56.3)
- moved F1 74.8 mm to (124.2, 114.5)
- moved R1 74.8 mm to (101.5, 102.0)
- moved R2 74.8 mm to (101.5, 105.0)
- moved R3 74.8 mm to (101.5, 108.0)
- moved R4 74.8 mm to (101.5, 110.9)
- moved R5 74.8 mm to (101.5, 113.8)
- moved R6 74.8 mm to (101.5, 116.8)
- moved C1 74.8 mm to (93.5, 98.0)
- moved C2 74.8 mm to (93.5, 101.0)
- moved C3 74.8 mm to (93.5, 104.0)
- moved C4 74.8 mm to (93.5, 107.0)
- moved C5 74.8 mm to (93.5, 110.0)
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
Commit message: Schematic rewrite maybe?
Parts:
- moved F1 85.0 mm to (108.0, 31.0)
- moved R6 83.9 mm to (97.5, 33.0), turned to 180 degrees
- moved R5 80.9 mm to (103.0, 33.0)
- moved C5 62.3 mm to (67.5, 53.5), turned to 90 degrees
- moved R3 61.6 mm to (66.1, 57.5), turned to 180 degrees
- moved C4 60.9 mm to (64.5, 53.5), turned to 90 degrees
- moved R2 56.8 mm to (66.1, 60.5), turned to 180 degrees
- moved C2 54.8 mm to (73.5, 50.0)
- moved J15 49.5 mm to (176.5, 30.0)
- moved J21 49.5 mm to (176.5, 42.5)
- moved J25 49.5 mm to (176.5, 55.5)
- moved J10 46.5 mm to (133.0, 33.0)
- moved J11 46.5 mm to (143.0, 23.0)
- moved J12 46.5 mm to (148.0, 33.0)
- moved J13 46.5 mm to (158.0, 23.0)
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
Commit message: Reworking stuffs
reworking schematic whilst tracing the PCB at the same time how fun!!!!
Parts:
- moved J24 114.5 mm to (135.0, 80.4)
- moved J4 114.5 mm to (147.0, 46.9)
- moved J5 114.5 mm to (136.0, 46.9)
- moved J8 114.5 mm to (145.0, 64.4)
- moved J16 99.8 mm to (153.2, 95.0)
- moved J17 99.8 mm to (158.2, 85.0)
- moved J2 99.8 mm to (143.2, 85.0)
- moved J3 99.8 mm to (128.2, 85.0)
- moved J6 99.8 mm to (138.2, 95.0)
- moved J7 99.8 mm to (123.2, 95.0)
- moved J21 74.2 mm to (102.5, 48.5), turned to -90 degrees
- moved J20 71.7 mm to (94.5, 48.5), turned to -90 degrees
- moved J23 64.3 mm to (102.5, 74.0), turned to -90 degrees
- moved J29 64.2 mm to (102.5, 60.0), turned to -90 degrees
- moved J22 61.7 mm to (94.5, 74.0), turned to -90 degrees
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Connections:
- J10 pad 1: Net-(J10-Pin_1) -> unconnected-(J10-Pin_1-Pad1)
- J10 pad 2: Net-(J10-Pin_2) -> unconnected-(J10-Pin_2-Pad2)
- J11 pad 1: Net-(J11-Pin_1) -> unconnected-(J11-Pin_1-Pad1)
- J11 pad 2: Net-(J11-Pin_2) -> unconnected-(J11-Pin_2-Pad2)
- J12 pad 1: Net-(J12-Pin_1) -> unconnected-(J12-Pin_1-Pad1)
- J12 pad 2: Net-(J12-Pin_2) -> unconnected-(J12-Pin_2-Pad2)
- J13 pad 1: Net-(J13-Pin_1) -> unconnected-(J13-Pin_1-Pad1)
- J13 pad 2: Net-(J13-Pin_2) -> unconnected-(J13-Pin_2-Pad2)
- J14 pad 1: Net-(J14-Pin_1) -> unconnected-(J14-Pin_1-Pad1)
- J14 pad 2: Net-(J14-Pin_2) -> unconnected-(J14-Pin_2-Pad2)
- J15 pad 1: Net-(J15-Pin_1) -> unconnected-(J15-Pin_1-Pad1)
- J15 pad 2: Net-(J15-Pin_2) -> unconnected-(J15-Pin_2-Pad2)
- J16 pad 1: Net-(J16-Pin_1) -> unconnected-(J16-Pin_1-Pad1)
- J16 pad 2: Net-(J16-Pin_2) -> unconnected-(J16-Pin_2-Pad2)
- J16 pad 3: GND -> unconnected-(J16-Pin_3-Pad3)
- J16 pad 4: GND -> unconnected-(J16-Pin_4-Pad4)
- J17 pad 1: Net-(J17-Pin_1) -> unconnected-(J17-Pin_1-Pad1)
- J17 pad 2: Net-(J17-Pin_2) -> unconnected-(J17-Pin_2-Pad2)
- J17 pad 3: GND -> unconnected-(J17-Pin_3-Pad3)
- J17 pad 4: GND -> unconnected-(J17-Pin_4-Pad4)
- J18 pad 1: PE0 -> unconnected-(J18-Pin_1-Pad1)
- J18 pad 2: PE1 -> unconnected-(J18-Pin_2-Pad2)
- J18 pad 3: GND -> unconnected-(J18-Pin_3-Pad3)
- J18 pad 4: GND -> unconnected-(J18-Pin_4-Pad4)
- J19 pad 1: PE3 -> unconnected-(J19-Pin_1-Pad1)
- J19 pad 2: PE4 -> unconnected-(J19-Pin_2-Pad2)
- J19 pad 3: GND -> unconnected-(J19-Pin_3-Pad3)
- J19 pad 4: GND -> unconnected-(J19-Pin_4-Pad4)
- J2 pad 1: Net-(J2-Pin_1) -> unconnected-(J2-Pin_1-Pad1)
- J2 pad 2: Net-(J2-Pin_2) -> unconnected-(J2-Pin_2-Pad2)
- J20 pad 1: +5V -> PF0
- J20 pad 2: PF0 -> unconnected-(J20-Pin_2-Pad2)
- J20 pad 3: GND -> unconnected-(J20-Pin_3-Pad3)
- J21 pad 1: +5V -> PF1
- J21 pad 2: PF1 -> unconnected-(J21-Pin_2-Pad2)
- J21 pad 3: GND -> unconnected-(J21-Pin_3-Pad3)
- J22 pad 1: +5V -> unconnected-(J22-Pin_1-Pad1)
- J22 pad 2: PE5 -> unconnected-(J22-Pin_2-Pad2)
- J22 pad 3: GND -> unconnected-(J22-Pin_3-Pad3)
- J23 pad 1: +5V -> unconnected-(J23-Pin_1-Pad1)
- J23 pad 2: PE6 -> unconnected-(J23-Pin_2-Pad2)
- J23 pad 3: GND -> unconnected-(J23-Pin_3-Pad3)
- J24 pad 1: +5V -> unconnected-(J24-Pin_1-Pad1)
- J24 pad 2: PE7 -> unconnected-(J24-Pin_2-Pad2)
- J24 pad 3: GND -> unconnected-(J24-Pin_3-Pad3)
- J25 pad 1: +5V -> unconnected-(J25-Pin_1-Pad1)
- J25 pad 2: PF6 -> unconnected-(J25-Pin_2-Pad2)
- J25 pad 3: GND -> unconnected-(J25-Pin_3-Pad3)
- J26 pad 1: +5V -> unconnected-(J26-Pin_1-Pad1)
- J26 pad 2: PF7 -> unconnected-(J26-Pin_2-Pad2)
- J26 pad 3: GND -> unconnected-(J26-Pin_3-Pad3)
- J28 pad 1: +5V -> PF2
- J28 pad 2: PF2 -> PF3
- J28 pad 3: PF3 -> unconnected-(J28-Pin_3-Pad3)
- J28 pad 4: GND -> unconnected-(J28-Pin_4-Pad4)
- J29 pad 1: +5V -> PF4
- J29 pad 2: PF4 -> PF5
- J29 pad 3: PF5 -> unconnected-(J29-Pin_3-Pad3)
- J29 pad 4: GND -> unconnected-(J29-Pin_4-Pad4)
- J3 pad 1: Net-(J3-Pin_1) -> unconnected-(J3-Pin_1-Pad1)
- J3 pad 2: Net-(J3-Pin_2) -> unconnected-(J3-Pin_2-Pad2)
- J4 pad 1: Net-(J4-Pin_1) -> unconnected-(J4-Pin_1-Pad1)
- J4 pad 2: Net-(J4-Pin_2) -> unconnected-(J4-Pin_2-Pad2)
- J5 pad 1: Net-(J5-Pin_1) -> unconnected-(J5-Pin_1-Pad1)
- J5 pad 2: Net-(J5-Pin_2) -> unconnected-(J5-Pin_2-Pad2)
- J6 pad 1: Net-(J6-Pin_1) -> unconnected-(J6-Pin_1-Pad1)
- J6 pad 2: Net-(J6-Pin_2) -> unconnected-(J6-Pin_2-Pad2)
- J7 pad 1: Net-(J7-Pin_1) -> unconnected-(J7-Pin_1-Pad1)
- J7 pad 2: Net-(J7-Pin_2) -> unconnected-(J7-Pin_2-Pad2)
- J8 pad 1: Net-(J8-Pin_1) -> unconnected-(J8-Pin_1-Pad1)
- J8 pad 2: Net-(J8-Pin_2) -> unconnected-(J8-Pin_2-Pad2)
- J9 pad 1: Net-(J9-Pin_1) -> unconnected-(J9-Pin_1-Pad1)
- J9 pad 2: Net-(J9-Pin_2) -> unconnected-(J9-Pin_2-Pad2)
- U1 pad 1: PE6 -> unconnected-(U1-PE6-Pad1)
- U1 pad 10: Net-(J6-Pin_1) -> unconnected-(U1-PB0-Pad10)
- U1 pad 11: Net-(J6-Pin_2) -> unconnected-(U1-PB1-Pad11)
- U1 pad 12: Net-(J7-Pin_1) -> unconnected-(U1-PB2-Pad12)
- U1 pad 13: Net-(J7-Pin_2) -> unconnected-(U1-PB3-Pad13)
- U1 pad 14: Net-(J8-Pin_1) -> unconnected-(U1-PB4-Pad14)
- U1 pad 15: Net-(J8-Pin_2) -> unconnected-(U1-PB5-Pad15)
- U1 pad 16: Net-(J9-Pin_1) -> unconnected-(U1-PB6-Pad16)
- U1 pad 17: Net-(J9-Pin_2) -> unconnected-(U1-PB7-Pad17)
- U1 pad 19: PE5 -> unconnected-(U1-PE5-Pad19)
- U1 pad 2: PE7 -> unconnected-(U1-PE7-Pad2)
- U1 pad 25: Net-(J12-Pin_1) -> unconnected-(U1-PD0-Pad25)
- U1 pad 26: Net-(J12-Pin_2) -> unconnected-(U1-PD1-Pad26)
- U1 pad 27: Net-(J14-Pin_1) -> unconnected-(U1-PD2-Pad27)
- U1 pad 28: Net-(J14-Pin_2) -> unconnected-(U1-PD3-Pad28)
- U1 pad 29: Net-(J16-Pin_1) -> unconnected-(U1-PD4-Pad29)
- U1 pad 30: Net-(J16-Pin_2) -> unconnected-(U1-PD5-Pad30)
- U1 pad 31: Net-(J17-Pin_1) -> unconnected-(U1-PD6-Pad31)
- U1 pad 32: Net-(J17-Pin_2) -> unconnected-(U1-PD7-Pad32)
- U1 pad 35: Net-(J11-Pin_1) -> unconnected-(U1-PC0-Pad35)
- U1 pad 36: Net-(J11-Pin_2) -> unconnected-(U1-PC1-Pad36)
- U1 pad 37: Net-(J13-Pin_1) -> unconnected-(U1-PC2-Pad37)
- U1 pad 38: Net-(J13-Pin_2) -> unconnected-(U1-PC3-Pad38)
- U1 pad 39: Net-(J15-Pin_1) -> unconnected-(U1-PC4-Pad39)
- U1 pad 40: Net-(J15-Pin_2) -> unconnected-(U1-PC5-Pad40)
- U1 pad 41: Net-(J10-Pin_1) -> unconnected-(U1-PC6-Pad41)
- U1 pad 42: Net-(J10-Pin_2) -> unconnected-(U1-PC7-Pad42)
- U1 pad 44: Net-(J5-Pin_2) -> unconnected-(U1-PA7-Pad44)
- U1 pad 45: Net-(J5-Pin_1) -> unconnected-(U1-PA6-Pad45)
- U1 pad 46: Net-(J4-Pin_2) -> unconnected-(U1-PA5-Pad46)
- U1 pad 47: Net-(J4-Pin_1) -> unconnected-(U1-PA4-Pad47)
- U1 pad 48: Net-(J3-Pin_2) -> unconnected-(U1-PA3-Pad48)
- U1 pad 49: Net-(J3-Pin_1) -> unconnected-(U1-PA2-Pad49)
- U1 pad 50: Net-(J2-Pin_2) -> unconnected-(U1-PA1-Pad50)
- U1 pad 51: Net-(J2-Pin_1) -> unconnected-(U1-PA0-Pad51)
Routing:
- net PF4: track 0.00 -> 36.0 mm
- net PF5: track 0.00 -> 34.1 mm
- net PF1: track 0.00 -> 33.1 mm
- net PF0: track 0.00 -> 24.7 mm
- net PF3: track 0.00 -> 21.1 mm
- net PF2: track 0.00 -> 20.6 mm
- net +5V: track 0.00 -> 10.5 mm
- net Net-(U1-UCAP): track 0.00 -> 5.88 mm
- net Net-(U1-D+): track 0.00 -> 3.51 mm
- net Net-(U1-D-): track 0.00 -> 3.18 mm

Commit message: I forgot to commit this oopsiedaisies
Parts:
- moved J25 95.1 mm to (97.5, 108.5), turned to 180 degrees
- moved J26 80.0 mm to (97.4, 80.0), turned to 180 degrees
- moved J23 44.3 mm to (97.5, 118.0), turned to 180 degrees
- moved J24 38.6 mm to (97.5, 89.5), turned to 180 degrees
- moved J22 25.2 mm to (97.4, 99.0), turned to 180 degrees
- moved R1 1.90 mm to (68.5, 74.0)
- moved C3 1.73 mm to (55.0, 56.5)
Connections:
- J22 pad 1: unconnected-(J22-Pin_1-Pad1) -> PA0
- J23 pad 1: unconnected-(J23-Pin_1-Pad1) -> PA2
- J24 pad 1: unconnected-(J24-Pin_1-Pad1) -> PF7
- J25 pad 1: unconnected-(J25-Pin_1-Pad1) -> PA1
- J26 pad 1: unconnected-(J26-Pin_1-Pad1) -> PF6
- U1 pad 49: unconnected-(U1-PA2-Pad49) -> PA2
- U1 pad 50: unconnected-(U1-PA1-Pad50) -> PA1
- U1 pad 51: unconnected-(U1-PA0-Pad51) -> PA0
Routing:
- net PF4: track 36.0 -> 0.00 mm
- net PF5: track 34.1 -> 0.00 mm
- net PF1: track 33.1 -> 0.00 mm
- net PF0: track 24.7 -> 0.00 mm
- net PF3: track 21.1 -> 0.00 mm
- net PF2: track 20.6 -> 0.42 mm
- net +5V: track 10.5 -> 2.95 mm

Commit message: AAAAAAAA
Parts:
- J24: value LED P1 Buttons -> LED P1 Console
- J25: value LED P2 Buttons -> LED P2 Console
- moved J22 127.3 mm to (224.3, 88.5)
- moved J23 127.3 mm to (224.4, 107.5)
- moved J24 127.3 mm to (224.4, 79.0)
- moved J25 127.3 mm to (224.4, 98.0)
- moved J26 127.3 mm to (224.3, 69.5)
- moved J20 98.2 mm to (192.5, 54.1)
- moved J21 98.2 mm to (200.5, 54.1)
- moved J28 98.2 mm to (192.5, 65.6)
- moved J29 98.2 mm to (200.5, 65.6)
- moved R1 0.50 mm to (68.0, 74.0)
Connections:
- J10 pad 1: unconnected-(J10-Pin_1-Pad1) -> PC1
- J10 pad 2: unconnected-(J10-Pin_2-Pad2) -> PC0
- J10 pad 3: GND -> unconnected-(J10-Pin_3-Pad3)
- J10 pad 4: GND -> unconnected-(J10-Pin_4-Pad4)
- J11 pad 1: unconnected-(J11-Pin_1-Pad1) -> PE1
- J11 pad 2: unconnected-(J11-Pin_2-Pad2) -> PE0
- J11 pad 3: GND -> unconnected-(J11-Pin_3-Pad3)
- J11 pad 4: GND -> unconnected-(J11-Pin_4-Pad4)
- J12 pad 1: unconnected-(J12-Pin_1-Pad1) -> PD7
- J12 pad 2: unconnected-(J12-Pin_2-Pad2) -> PD6
- J12 pad 3: GND -> unconnected-(J12-Pin_3-Pad3)
- J12 pad 4: GND -> unconnected-(J12-Pin_4-Pad4)
- J13 pad 1: unconnected-(J13-Pin_1-Pad1) -> PD5
- J13 pad 2: unconnected-(J13-Pin_2-Pad2) -> PD4
- J13 pad 3: GND -> unconnected-(J13-Pin_3-Pad3)
- J13 pad 4: GND -> unconnected-(J13-Pin_4-Pad4)
- J14 pad 1: unconnected-(J14-Pin_1-Pad1) -> PD3
- J14 pad 2: unconnected-(J14-Pin_2-Pad2) -> PD2
- J14 pad 3: GND -> unconnected-(J14-Pin_3-Pad3)
- J14 pad 4: GND -> unconnected-(J14-Pin_4-Pad4)
- J15 pad 1: unconnected-(J15-Pin_1-Pad1) -> PD1
- J15 pad 2: unconnected-(J15-Pin_2-Pad2) -> PD0
- J15 pad 3: GND -> unconnected-(J15-Pin_3-Pad3)
- J15 pad 4: GND -> unconnected-(J15-Pin_4-Pad4)
- J16 pad 1: unconnected-(J16-Pin_1-Pad1) -> PE5
- J16 pad 2: unconnected-(J16-Pin_2-Pad2) -> PE4
- J17 pad 1: unconnected-(J17-Pin_1-Pad1) -> PB7
- J17 pad 2: unconnected-(J17-Pin_2-Pad2) -> PB6
- J18 pad 1: unconnected-(J18-Pin_1-Pad1) -> PB5
- J18 pad 2: unconnected-(J18-Pin_2-Pad2) -> PB4
- J19 pad 1: unconnected-(J19-Pin_1-Pad1) -> PB3
- J19 pad 2: unconnected-(J19-Pin_2-Pad2) -> PB2
- J2 pad 1: unconnected-(J2-Pin_1-Pad1) -> PF6
- J2 pad 2: unconnected-(J2-Pin_2-Pad2) -> PF7
- J2 pad 3: GND -> unconnected-(J2-Pin_3-Pad3)
- J2 pad 4: GND -> unconnected-(J2-Pin_4-Pad4)
- J22 pad 1: PA0 -> PE7
- J23 pad 1: PA2 -> PE6
- J24 pad 1: PF7 -> PB0
- J25 pad 1: PA1 -> PE3
- J26 pad 1: PF6 -> PB1
- J3 pad 1: unconnected-(J3-Pin_1-Pad1) -> PA2
- J3 pad 2: unconnected-(J3-Pin_2-Pad2) -> PA3
- J3 pad 3: GND -> unconnected-(J3-Pin_3-Pad3)
- J3 pad 4: GND -> unconnected-(J3-Pin_4-Pad4)
- J4 pad 1: unconnected-(J4-Pin_1-Pad1) -> PA6
- J4 pad 2: unconnected-(J4-Pin_2-Pad2) -> PA7
- J4 pad 3: GND -> unconnected-(J4-Pin_3-Pad3)
- J4 pad 4: GND -> unconnected-(J4-Pin_4-Pad4)
- J5 pad 1: unconnected-(J5-Pin_1-Pad1) -> PC5
- J5 pad 2: unconnected-(J5-Pin_2-Pad2) -> PC4
- J5 pad 3: GND -> unconnected-(J5-Pin_3-Pad3)
- J5 pad 4: GND -> unconnected-(J5-Pin_4-Pad4)
- J6 pad 1: unconnected-(J6-Pin_1-Pad1) -> PA0
- J6 pad 2: unconnected-(J6-Pin_2-Pad2) -> PA1
- J6 pad 3: GND -> unconnected-(J6-Pin_3-Pad3)
- J6 pad 4: GND -> unconnected-(J6-Pin_4-Pad4)
- J7 pad 1: unconnected-(J7-Pin_1-Pad1) -> PA4
- J7 pad 2: unconnected-(J7-Pin_2-Pad2) -> PA5
- J7 pad 3: GND -> unconnected-(J7-Pin_3-Pad3)
- J7 pad 4: GND -> unconnected-(J7-Pin_4-Pad4)
- J8 pad 1: unconnected-(J8-Pin_1-Pad1) -> PC7
- J8 pad 2: unconnected-(J8-Pin_2-Pad2) -> PC6
- J8 pad 3: GND -> unconnected-(J8-Pin_3-Pad3)
- J8 pad 4: GND -> unconnected-(J8-Pin_4-Pad4)
- J9 pad 1: unconnected-(J9-Pin_1-Pad1) -> PC3
- J9 pad 2: unconnected-(J9-Pin_2-Pad2) -> PC2
- J9 pad 3: GND -> unconnected-(J9-Pin_3-Pad3)
- J9 pad 4: GND -> unconnected-(J9-Pin_4-Pad4)
- U1 pad 1: unconnected-(U1-PE6-Pad1) -> PE6
- U1 pad 10: unconnected-(U1-PB0-Pad10) -> PB0
- U1 pad 11: unconnected-(U1-PB1-Pad11) -> PB1
- U1 pad 12: unconnected-(U1-PB2-Pad12) -> PB2
- U1 pad 13: unconnected-(U1-PB3-Pad13) -> PB3
- U1 pad 14: unconnected-(U1-PB4-Pad14) -> PB4
- U1 pad 15: unconnected-(U1-PB5-Pad15) -> PB5
- U1 pad 16: unconnected-(U1-PB6-Pad16) -> PB6
- U1 pad 17: unconnected-(U1-PB7-Pad17) -> PB7
- U1 pad 19: unconnected-(U1-PE5-Pad19) -> PE5
- U1 pad 2: unconnected-(U1-PE7-Pad2) -> PE7
- U1 pad 25: unconnected-(U1-PD0-Pad25) -> PD0
- U1 pad 26: unconnected-(U1-PD1-Pad26) -> PD1
- U1 pad 27: unconnected-(U1-PD2-Pad27) -> PD2
- U1 pad 28: unconnected-(U1-PD3-Pad28) -> PD3
- U1 pad 29: unconnected-(U1-PD4-Pad29) -> PD4
- U1 pad 30: unconnected-(U1-PD5-Pad30) -> PD5
- U1 pad 31: unconnected-(U1-PD6-Pad31) -> PD6
- U1 pad 32: unconnected-(U1-PD7-Pad32) -> PD7
- U1 pad 35: unconnected-(U1-PC0-Pad35) -> PC0
- U1 pad 36: unconnected-(U1-PC1-Pad36) -> PC1
- U1 pad 37: unconnected-(U1-PC2-Pad37) -> PC2
- U1 pad 38: unconnected-(U1-PC3-Pad38) -> PC3
- U1 pad 39: unconnected-(U1-PC4-Pad39) -> PC4
- U1 pad 40: unconnected-(U1-PC5-Pad40) -> PC5
- U1 pad 41: unconnected-(U1-PC6-Pad41) -> PC6
- U1 pad 42: unconnected-(U1-PC7-Pad42) -> PC7
- U1 pad 44: unconnected-(U1-PA7-Pad44) -> PA7
- U1 pad 45: unconnected-(U1-PA6-Pad45) -> PA6
- U1 pad 46: unconnected-(U1-PA5-Pad46) -> PA5
- U1 pad 47: unconnected-(U1-PA4-Pad47) -> PA4
- U1 pad 48: unconnected-(U1-PA3-Pad48) -> PA3

Commit message: Death.
Parts:
- C2, C3, C4: value 0.1uf -> 1uf
- moved J23 223.0 mm to (21.1, 16.1), turned to -90 degrees
- moved J22 212.3 mm to (21.0, 27.3), turned to -90 degrees
- moved J25 207.2 mm to (20.5, 60.8), turned to -90 degrees
- moved J24 206.0 mm to (20.6, 49.5), turned to -90 degrees
- moved J26 204.0 mm to (20.3, 71.9), turned to -90 degrees
- moved J20 162.6 mm to (33.6, 20.0), turned to 180 degrees
- moved J21 159.5 mm to (44.7, 19.9), turned to 180 degrees
- moved J28 141.1 mm to (59.0, 19.9), turned to 180 degrees
- moved J29 135.8 mm to (72.6, 19.9), turned to 180 degrees
- moved J17 124.7 mm to (36.0, 60.3), turned to 180 degrees
- moved J13 107.2 mm to (65.2, 76.7), turned to 90 degrees
- moved J15 103.4 mm to (84.3, 76.7)
- moved J14 102.4 mm to (74.9, 76.7), turned to 90 degrees
- moved J2 92.4 mm to (65.2, 35.4), turned to 90 degrees
- moved J18 89.9 mm to (36.0, 69.5), turned to 180 degrees
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Connections:
- J10 pad 1: PC1 -> PE1
- J10 pad 2: PC0 -> PE0
- J10 pad 3: unconnected-(J10-Pin_3-Pad3) -> GND
- J10 pad 4: unconnected-(J10-Pin_4-Pad4) -> GND
- J11 pad 1: PE1 -> PD7
- J11 pad 2: PE0 -> PD6
- J11 pad 3: unconnected-(J11-Pin_3-Pad3) -> GND
- J11 pad 4: unconnected-(J11-Pin_4-Pad4) -> GND
- J12 pad 1: PD7 -> PD5
- J12 pad 2: PD6 -> PD4
- J12 pad 3: unconnected-(J12-Pin_3-Pad3) -> GND
- J12 pad 4: unconnected-(J12-Pin_4-Pad4) -> GND
- J13 pad 1: PD5 -> PD3
- J13 pad 2: PD4 -> PD2
- J13 pad 3: unconnected-(J13-Pin_3-Pad3) -> GND
- J13 pad 4: unconnected-(J13-Pin_4-Pad4) -> GND
- J14 pad 1: PD3 -> PD1
- J14 pad 2: PD2 -> PD0
- J14 pad 3: unconnected-(J14-Pin_3-Pad3) -> GND
- J14 pad 4: unconnected-(J14-Pin_4-Pad4) -> GND
- J15 pad 1: PD1 -> PE5
- J15 pad 2: PD0 -> PE4
- J15 pad 3: unconnected-(J15-Pin_3-Pad3) -> GND
- J15 pad 4: unconnected-(J15-Pin_4-Pad4) -> GND
- J16 pad 1: PE5 -> PC2
- J16 pad 2: PE4 -> PC3
- J16 pad 3: unconnected-(J16-Pin_3-Pad3) -> GND
- J16 pad 4: unconnected-(J16-Pin_4-Pad4) -> GND
- J17 pad 3: unconnected-(J17-Pin_3-Pad3) -> GND
- J17 pad 4: unconnected-(J17-Pin_4-Pad4) -> GND
- J18 pad 3: unconnected-(J18-Pin_3-Pad3) -> GND
- J18 pad 4: unconnected-(J18-Pin_4-Pad4) -> GND
- J19 pad 3: unconnected-(J19-Pin_3-Pad3) -> GND
- J19 pad 4: unconnected-(J19-Pin_4-Pad4) -> GND
- J2 pad 1: PF6 -> PF7
- J2 pad 2: PF7 -> PF6
- J2 pad 3: unconnected-(J2-Pin_3-Pad3) -> GND
- J2 pad 4: unconnected-(J2-Pin_4-Pad4) -> GND
- J20 pad 2: unconnected-(J20-Pin_2-Pad2) -> +5V
- J20 pad 3: unconnected-(J20-Pin_3-Pad3) -> GND
- J21 pad 2: unconnected-(J21-Pin_2-Pad2) -> +5V
- J21 pad 3: unconnected-(J21-Pin_3-Pad3) -> GND
- J22 pad 2: unconnected-(J22-Pin_2-Pad2) -> +5V
- J22 pad 3: unconnected-(J22-Pin_3-Pad3) -> GND
- J23 pad 2: unconnected-(J23-Pin_2-Pad2) -> +5V
- J23 pad 3: unconnected-(J23-Pin_3-Pad3) -> GND
- J24 pad 1: PB0 -> PE3
- J24 pad 2: unconnected-(J24-Pin_2-Pad2) -> +5V
- J24 pad 3: unconnected-(J24-Pin_3-Pad3) -> GND
- J25 pad 1: PE3 -> PB0
- J25 pad 2: unconnected-(J25-Pin_2-Pad2) -> +5V
- J25 pad 3: unconnected-(J25-Pin_3-Pad3) -> GND
- J26 pad 2: unconnected-(J26-Pin_2-Pad2) -> +5V
- J26 pad 3: unconnected-(J26-Pin_3-Pad3) -> GND
- J28 pad 3: unconnected-(J28-Pin_3-Pad3) -> +5V
- J28 pad 4: unconnected-(J28-Pin_4-Pad4) -> GND
- J29 pad 3: unconnected-(J29-Pin_3-Pad3) -> +5V
- J29 pad 4: unconnected-(J29-Pin_4-Pad4) -> GND
- J3 pad 1: PA2 -> PA3
- J3 pad 2: PA3 -> PA2
- J3 pad 3: unconnected-(J3-Pin_3-Pad3) -> GND
- J3 pad 4: unconnected-(J3-Pin_4-Pad4) -> GND
- J4 pad 1: PA6 -> PA7
- J4 pad 2: PA7 -> PA6
- J4 pad 3: unconnected-(J4-Pin_3-Pad3) -> GND
- J4 pad 4: unconnected-(J4-Pin_4-Pad4) -> GND
- J5 pad 1: PC5 -> PC4
- J5 pad 2: PC4 -> PC5
- J5 pad 3: unconnected-(J5-Pin_3-Pad3) -> GND
- J5 pad 4: unconnected-(J5-Pin_4-Pad4) -> GND
- J6 pad 1: PA0 -> PA1
- J6 pad 2: PA1 -> PA0
- J6 pad 3: unconnected-(J6-Pin_3-Pad3) -> GND
- J6 pad 4: unconnected-(J6-Pin_4-Pad4) -> GND
- J7 pad 1: PA4 -> PA5
- J7 pad 2: PA5 -> PA4
- J7 pad 3: unconnected-(J7-Pin_3-Pad3) -> GND
- J7 pad 4: unconnected-(J7-Pin_4-Pad4) -> GND
- J8 pad 1: PC7 -> PC6
- J8 pad 2: PC6 -> PC7
- J8 pad 3: unconnected-(J8-Pin_3-Pad3) -> GND
- J8 pad 4: unconnected-(J8-Pin_4-Pad4) -> GND
- J9 pad 1: PC3 -> PC1
- J9 pad 2: PC2 -> PC0
- J9 pad 3: unconnected-(J9-Pin_3-Pad3) -> GND
- J9 pad 4: unconnected-(J9-Pin_4-Pad4) -> GND
Routing:
- net GND: track 0.00 -> 97.8 mm
- net +5V: track 2.95 -> 74.8 mm, vias 0 -> 3
- net Net-(U1-XTAL2): track 0.00 -> 15.0 mm
- net Net-(U1-XTAL1): track 0.05 -> 13.6 mm
- net D-: track 0.00 -> 12.0 mm
- net D+: track 0.00 -> 12.0 mm
- net VCC: track 0.00 -> 8.03 mm
- net Net-(U1-D-): track 3.18 -> 9.46 mm
- net Net-(U1-D+): track 3.51 -> 9.13 mm
- net CC1: track 0.00 -> 4.11 mm
- net Net-(U1-~{RESET}): track 0.00 -> 3.54 mm
- net Net-(U1-UCAP): track 5.88 -> 3.30 mm
- net PC7: track 0.00 -> 2.28 mm
- net PA7: track 0.00 -> 2.20 mm
- net CC2: track 0.00 -> 2.17 mm
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Other:
- board outline added: 89.2 x 69.1 mm
- board text added: "Button 1"
- board text added: "Button 2"
- board text added: "Button 3"
- board text added: "Button 4"
- board text added: "Button 5"
- board text added: "Button 6"
- board text added: "Button 7"
- board text added: "Button LED Connectors"
- board text added: "Button Start"
- board text added: "Center Console"
- board text added: "Console Buttons"
- board text added: "EFFECT"
- board text added: "P1 Analog"
- board text added: "P1 Encoder"
- board text added: "P2 Analog"
- board text added: "P2 Encoder"
- board text added: "Player 1"
- board text added: "Player 1 Buttons"
- board text added: "Player 2"
- board text added: "Player 2 Buttons"
- board text added: "Turntable Connectors"
- board text added: "Turntable LED Connectors"
- board text added: "VEFX"

Commit message: Wha?
Parts:
- removed J1: USB_C_Receptacle_USB2.0_16P, Connector_USB:USB_C_Receptacle_HRO_TYPE-C-31-M-12
- removed R5, R6: 5k1, Resistor_SMD:R_0805_2012Metric
- added J27: USB Type C Connector, Connector_JST:JST_XH_B4B-XH-AM_1x04_P2.50mm_Vertical, F.Cu at (60.5, 49.8)
- moved J25 44.1 mm to (62.2, 75.1)
- moved J24 44.1 mm to (62.2, 63.8)
- moved J26 44.1 mm to (62.0, 86.2)
- moved C6 43.6 mm to (94.5, 73.6)
- moved C7 43.6 mm to (86.8, 73.5)
- moved Y1 43.6 mm to (90.7, 73.5)
- moved C4 43.6 mm to (85.5, 67.9)
- moved C3 43.4 mm to (93.3, 43.8)
- moved J14 43.2 mm to (116.5, 88.4)
- moved J13 43.2 mm to (106.8, 88.4)
- moved J15 43.2 mm to (125.9, 88.4)
- moved J19 43.2 mm to (135.4, 88.4)
- moved J12 43.1 mm to (135.4, 74.8)
- moved J11 43.1 mm to (125.9, 74.7)
- moved J10 43.1 mm to (116.5, 74.7)
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Connections:
- J10 pad 1: PE1 -> PE0
- J10 pad 2: PE0 -> PE1
- J11 pad 1: PD7 -> PD6
- J11 pad 2: PD6 -> PD7
- J12 pad 1: PD5 -> PD4
- J12 pad 2: PD4 -> PD5
- J13 pad 1: PD3 -> PD2
- J13 pad 2: PD2 -> PD3
- J14 pad 1: PD1 -> PD0
- J14 pad 2: PD0 -> PD1
- J15 pad 1: PE5 -> PE4
- J15 pad 2: PE4 -> PE5
- J17 pad 1: PB7 -> PB2
- J17 pad 2: PB6 -> PB3
- J18 pad 1: PB5 -> PB4
- J18 pad 2: PB4 -> PB5
- J19 pad 1: PB3 -> PB6
- J19 pad 2: PB2 -> PB7
- J28 pad 1: PF2 -> PF3
- J28 pad 2: PF3 -> PF2
- J29 pad 1: PF4 -> PF5
- J29 pad 2: PF5 -> PF4
- J9 pad 1: PC1 -> PC0
- J9 pad 2: PC0 -> PC1
Routing:
- net GND: track 97.8 -> 756.9 mm
- net +5V: track 74.8 -> 252.2 mm, vias 3 -> 6
- net PB6: track 0.00 -> 82.4 mm
- net PB7: track 0.00 -> 80.3 mm
- net PE5: track 0.00 -> 69.2 mm
- net PE4: track 0.00 -> 69.0 mm
- net PD4: track 0.00 -> 55.7 mm
- net PD5: track 0.00 -> 55.4 mm
- net PD0: track 0.00 -> 51.0 mm
- net PD1: track 0.00 -> 50.6 mm
- net PC3: track 0.00 -> 45.4 mm
- net PC2: track 0.00 -> 44.3 mm
- net PD6: track 0.00 -> 43.5 mm
- net PD7: track 0.00 -> 43.2 mm
- net PB1: track 0.74 -> 43.7 mm
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- added copper zone on B.Cu, net (none)
- added copper zone on F.Cu, net (none)
- added copper zone on B.Cu, net GND
- added copper zone on F.Cu, net GND
Other:
- board size 89.2 x 69.1 mm -> 97 x 74.4 mm
- board text added: "USB Connector"
