File: PHIIDXDP.kicad_pcb (KiCad board)
At the start: 2 copper layers, 97 x 74.4 mm, 43 parts, among them J10 2P BT 2, J11 2P BT 3, J12 2P BT 4, J13 2P BT 5, J14 2P BT 6, J15 2P BT 7, J16 1P START, J17 EFFECT, J18 VEFX, J19 2P START, J2 1P BT 1, J20 P1 TT analog, J21 P2 TT analog, J22 LED P1 TT, J23 LED P2 TT, J24 LED P1 Console, J25 LED P2 Console, J26 LED CENTER, J27 USB Type C Connector, J28 P1 TT Encoder, J29 P2 TT Encoder, J3 1P BT 3, J4 1P BT 5, J5 1P BT 7, J6 1P BT 2, J7 1P BT 4, J8 1P BT 6, J9 2P BT 1, SW1 SW_Push, U1 AT90USB647-A, Y1 16MHz

Commit message: No way!
Parts:
- moved J12 4.15 mm to (135.6, 78.9)
- moved C6 4.15 mm to (94.6, 77.8)
- moved J10 4.15 mm to (116.6, 78.9)
- moved J18 4.15 mm to (73.7, 79.5)
- moved J9 4.15 mm to (106.9, 78.9)
- moved C2 4.15 mm to (77.5, 60.5)
- moved J17 4.15 mm to (73.7, 66.1)
- moved J2 4.15 mm to (106.9, 50.6)
- moved J21 4.15 mm to (86.4, 35.1)
- moved J28 4.15 mm to (100.7, 35.1)
- moved J29 4.15 mm to (114.3, 35.1)
- moved J3 4.15 mm to (126.2, 50.7)
- moved J5 4.15 mm to (126.2, 64.4)
- moved J6 4.15 mm to (116.6, 50.6)
- moved J7 4.15 mm to (135.9, 50.6)
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Other:
- board size 97 x 74.4 mm -> 97 x 81.8 mm
- board text added: "LED Center"
- board text added: "LED P1 Buttons"
- board text added: "LED P1 TT"
- board text added: "LED P2 Buttons"
- board text added: "LED P2 TT"
- board text added: "P1 BT 1"
- board text added: "P1 BT 2"
- board text added: "P1 BT 3"
- board text added: "P1 BT 4"
- board text added: "P1 BT 5"
- board text added: "P1 BT 6"
- board text added: "P1 BT 7"
- board text added: "P1 START"
- board text added: "P1 TT Analog"
- board text added: "P1 TT Encoder"
- board text added: "P2 BT 1"
- board text added: "P2 BT 2"
- board text added: "P2 BT 3"
- board text added: "P2 BT 4"
- board text added: "P2 BT 5"
- board text added: "P2 BT 6"
- board text added: "P2 BT 7"
- board text added: "P2 START"
- board text added: "P2 TT Analog"
- board text added: "P2 TT Encoder"
- board text added: "RESET"
- board text removed: "Button 1"
- board text removed: "Button 2"
- board text removed: "Button 3"
- board text removed: "Button 4"
- board text removed: "Button 5"
- board text removed: "Button 6"
- board text removed: "Button 7"
- board text removed: "Button LED Connectors"
- board text removed: "Button Start"
- board text removed: "Center Console"
- board text removed: "Console Buttons"
- board text removed: "P1 Analog"
- board text removed: "P1 Encoder"
- board text removed: "P2 Analog"
- board text removed: "P2 Encoder"
- board text removed: "Player 1"
- board text removed: "Player 1 Buttons"
- board text removed: "Player 2"
- board text removed: "Player 2 Buttons"
- board text removed: "Turntable Connectors"
- board text removed: "Turntable LED Connectors"
